File: Motherboard Schematics/Automatic Presser/Automatic Presser.sch (KiCad schematic (older format))
At the start: 21 parts, among them J1 Barrel_Jack_Switch, M1 Stepper_Motor_bipolar, M2 Stepper_Motor_bipolar, M3 Motor_Servo, SW1 SW_DIP_x03, SW2 SW_DIP_x03, SW3 SW_Push_Dual_x2, U1 Arduino_Nano_R3, U2 LM7809_TO220, U3 LM7805_TO220

Commit message: Changes to schematics
Parts:
- U1: symbol arduino_nano_r3:Arduino_Nano_R3 -> Automatic-Presser-rescue:Arduino_Nano_R3-arduino_nano_r3
Connections:
- net A1_DIR: now also U1.29 (D11/MOSI); no longer U1.26 (D8)
- net A1_EN: now also U1.26 (D8); no longer U1.28 (D10)
- net A2_DIR: now also U1.30 (D12/MISO); no longer U1.23 (D5)
- net A2_EN: now also U1.1 (D13/SCK); no longer U1.25 (D7)
- net A2_STEP: now also U1.28 (D10); no longer U1.24 (D6)
Changed lines of the file:
@@
 $EndDescr
 $Comp
-L arduino_nano_r3:Arduino_Nano_R3 U1
+L Automatic-Presser-rescue:Arduino_Nano_R3-arduino_nano_r3 U1
 U 1 1 603AB668
 P 4000 3000
@@
 NoConn ~ 3050 2500
 NoConn ~ 4200 2000
-Text GLabel 4950 3350 2    50   Output ~ 0
+Text GLabel 4950 3150 2    50   Output ~ 0
 A1_EN
 Text GLabel 4950 3250 2    50   Output ~ 0
 A1_STEP
-Text GLabel 4950 3150 2    50   Output ~ 0
+Text GLabel 4950 3450 2    50   Output ~ 0
 A1_DIR
-Text GLabel 4950 3050 2    50   Output ~ 0
+Text GLabel 4950 3650 2    50   Output ~ 0
 A2_EN
-Text GLabel 4950 2950 2    50   Output ~ 0
+Text GLabel 4950 3350 2    50   Output ~ 0
 A2_STEP
-Text GLabel 4950 2850 2    50   Output ~ 0
+Text GLabel 4950 3550 2    50   Output ~ 0
 A2_DIR
 $Comp
